File: Hardware/testing/T-USB-Testing/programmer.kicad_sch (KiCad schematic)
At the start: 3 parts

Commit message: MSP debug pins tweaks
Connections:
- net SWD CLK RP renamed T_SBWTCK
- net SWD DAT RP renamed T_SBWTDIO
- net UART RP RXD renamed UART T RXD
- net UART RP TXD renamed UART T TXD
Changed lines of the file:
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@@
     (effects (font (size 1.27 1.27)) (justify right))
   )
-  (hierarchical_label "UART RP TXD" (shape input) (at 124.46 66.04 0)
+  (hierarchical_label "UART T TXD" (shape input) (at 124.46 66.04 0)
     (effects (font (size 1.27 1.27)) (justify left))
   )
@@
     (effects (font (size 1.27 1.27)) (justify right))
   )
-  (hierarchical_label "SWD DAT RP" (shape input) (at 52.07 78.74 180)
+  (hierarchical_label "T_SBWTDIO" (shape input) (at 52.07 78.74 180)
     (effects (font (size 1.27 1.27)) (justify right))
   )
@@
     (effects (font (size 1.27 1.27)) (justify right))
   )
-  (hierarchical_label "UART RP RXD" (shape input) (at 124.46 68.58 0)
+  (hierarchical_label "UART T RXD" (shape input) (at 124.46 68.58 0)
     (effects (font (size 1.27 1.27)) (justify left))
   )
-  (hierarchical_label "SWD CLK RP" (shape input) (at 53.34 76.2 180)
+  (hierarchical_label "T_SBWTCK" (shape input) (at 53.34 76.2 180)
     (effects (font (size 1.27 1.27)) (justify right))
   )
