File: Hardware/929/Faceboard/Faceboard.kicad_sch (KiCad schematic)
At the start: 5 parts, among them P1 UCM-P1-100DS-0.4V, P2 UCM-P2-100DS-0.4V

Commit message: Bob 929
Parts:
- C100, C101, C102: footprint Capacitor_SMD:C_1210_3225Metric -> Capacitor_SMD:C_0402_1005Metric
Connections:
- net PCIE_WAKE_B renamed M2B_PERST
- net SPARE2_20 renamed TOUCH_nINT
- net SYS_EX_nINT renamed PD_USBC_INT
Other:
- removed sheet NVMe SSD B+M connected
- added sheet Combi Camera (combi-camera.kicad_sch)
