File: Hardware/929/Faceboard/M2-T-USB.kicad_sch (KiCad schematic)
At the start: 37 parts, among them J3 Debug_4-2328724-5, P5 T-USB_PWRCTL-50, P6 T-USB_HIGH-SPEED-50, U10 CBTL04083ABS_518, U11 TS5USBC410YFFR, U12 Faceboard_Expander_FR2032IG56, U13 PCA9555PW, U14 74HC595PW_118, U15 74HC595PW_118, U3 SN74CB3Q3245PW

Commit message: Bob 929
Parts:
- removed C115, C117, C118, C119, C120: 100nF, Capacitor_SMD:C_1210_3225Metric, symbol Device:C
- removed C116: 1uF, Capacitor_SMD:C_1210_3225Metric, symbol Device:C
- removed R10: 10K, Resistor_SMD:R_1206_3216Metric, symbol Device:R
- removed U13: PCA9555PW, Package_SO:TSSOP-24_4.4x7.8mm_P0.65mm, symbol Interface_Expansion:PCA9555PW
- C121, C122, C123, C124, C125: footprint Capacitor_SMD:C_1210_3225Metric -> Capacitor_SMD:C_0402_1005Metric
- R11: footprint Resistor_SMD:R_1206_3216Metric -> Resistor_SMD:R_0402_1005Metric
- U11: footprint Package_BGA:Texas_DSBGA-12_1.36x1.86mm_Layout3x4_P0.5mm -> Ziloo:TS5USBC410YFFR
- U3: value SN74CB3Q3245PW -> SN74CB3Q3245RGYR; footprint Ziloo:SN74CB3Q3245PW -> Ziloo:SN74CB3Q3245RGYR
Connections:
- net LEFT_ATT_XSHUT: no longer U14.3 (Q3)
- net LEFT_PWRDN: no longer U14.15 (Q0)
- net LEFT_RESET: no longer U14.1 (Q1)
- net RIGHT_ATT_XSHUT: no longer U14.7 (Q7)
- net RIGHT_PWRDN: no longer U14.4 (Q4)
- net RIGHT_RESET: no longer U14.5 (Q5)
- net BOTH_VSOM: now reaches U12.39 (BOTH_VSOM/P2.3)
- net BOTH_VSOM: now also P5.11 (BOTH_VSOM)
- net PD_USBC_INT: now reaches P5.38 (MIC_INT)
- net LEFT_ATT_INT: no longer names the net of U14.2 (Q2)
- net RIGHT_ATT_INT: no longer names the net of U14.6 (Q6)
Other:
- note added: "assign FACE EX pin"
- note added: "connect OE"
- note removed: "1.8V convert optional? both in parallel? with OE"
- note removed: "Micro SD socket?"
- note removed: "SYS I2C Address: 0x20"
- note removed: "Sound hookup 909c ?"
