File: Hardware/929/Faceboard/m2-key-b.kicad_sch (KiCad schematic)
At the start: 25 parts, among them Q1 2SC4213, U16 TXS0104EDR, U17 TXS0104EDR, U18 SN74CB3Q3245PW, U6 Supervisor M2 10128793-001RLF, Y1 25.000MHz

Commit message: Bob 929
Parts:
- removed U16, U17: TXS0104EDR, Ziloo:TXS0104EDR, symbol Ziloo:TXS0104EDR
- added U16, U17: TXS0104, Ziloo:TXS0104EYZTR, symbol Ziloo:TXS0104EYZTR
- C129, C130, C131, C132, C133, C134, C135, C136, C137, C138, C139, C141, C142, C143: footprint Capacitor_SMD:C_1210_3225Metric -> Capacitor_SMD:C_0402_1005Metric
- R12, R13, R14, R15, R16: footprint Resistor_SMD:R_1206_3216Metric -> Resistor_SMD:R_0402_1005Metric
- U18: value SN74CB3Q3245PW -> SN74CB3Q3245RGYR; footprint Ziloo:SN74CB3Q3245PW -> Ziloo:SN74CB3Q3245RGYR
Connections:
- net +1V8: now also U16.B1 (VCCB), U17.B1 (VCCB)
- net +3.3V: now also U16.B2 (VCCA), U17.B2 (VCCA)
- net B_OE_STEM: now also U17.B3 (OE)
- net B_OE_UART: now also U16.B3 (OE)
- net COEX: now also U16.C2 (B2)
- net GND: now also U16.D2 (GND), U17.D2 (GND)
- net GNSS_IRQ_3V3: now also U17.C3 (B3)
- net M2B_UART_RXD: now also U16.D1 (B4)
- net M2B_UART_TXD: now also U16.C3 (B3)
- net STEM_I2C_SCL: now also U17.C1 (B1)
- net STEM_I2C_SDA: now also U17.C2 (B2)
- net at U6.40 (STEM_SCL): now also U17.A1
- net at U6.42 (STEM_SDA): now also U17.A2
- net at U6.44 (GNSS_IRQ): now also U17.A3
- net at U6.46 (GPIO_3): now also U17.D3 (A4)
- net at U6.48 (GPIO_4): now also U16.A1
- net at U6.60 (COEX3): now also U16.A2
- net at U6.62 (M2B_UART_TXD): now also U16.A3
- net at U6.64 (M2B_UART_RXD): now also U16.D3 (A4)
