File: Hardware/929/Faceboard/using-ssd.kicad_sch (KiCad schematic)
At the start: 3 parts, among them U1 10128793-001RLF

Commit message: Bob 929
Parts:
- C1, C126: footprint Capacitor_SMD:C_1210_3225Metric -> Capacitor_SMD:C_0402_1005Metric
Changed lines of the file:
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@@
       (effects (font (size 1.27 1.27)) (justify left))
     )
-    (property "Footprint" "Capacitor_SMD:C_1210_3225Metric" (id 2) (at 198.12 59.69 0)
+    (property "Footprint" "Capacitor_SMD:C_0402_1005Metric" (id 2) (at 198.12 59.69 0)
       (effects (font (size 1.27 1.27)) hide)
     )
@@
       (effects (font (size 1.27 1.27)) (justify left))
     )
-    (property "Footprint" "Capacitor_SMD:C_1210_3225Metric" (id 2) (at 196.85 143.51 0)
+    (property "Footprint" "Capacitor_SMD:C_0402_1005Metric" (id 2) (at 196.85 143.51 0)
       (effects (font (size 1.27 1.27)) hide)
     )
